File: hardware/Handle/nyantern.kicad_pcb (KiCad board)
At the start: 2 copper layers, 49.6 x 97.2 mm, 0 parts

Commit message: God knows but a lot has changed
Routing:
- removed copper zone on F.Cu, net (none)
Changed lines of the file:
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@@
       (drillshape 0)
       (scaleselection 1)
-      (outputdirectory "Gerbers/"))
+      (outputdirectory "Gerbers - Handle V1/"))
   )
   (net 0 "")
@@
     (uvia_drill 0.1)
   )
+  (gr_line (start 165.8 53) (end 165.8 51.4) (layer Edge.Cuts) (width 0.05))
   (gr_line (start 130.8 121.2) (end 129.2 121.2) (layer Edge.Cuts) (width 0.05))
   (gr_line (start 172.8 79.2) (end 171.2 79.2) (layer Edge.Cuts) (width 0.05))
@@
   (gr_line (start 125.2 147) (end 134.2 147) (layer Edge.Cuts) (width 0.05))
   (gr_line (start 165.8 53) (end 174.8 53) (layer Edge.Cuts) (width 0.05))
-  (gr_line (start 165.8 51.4) (end 165.8 53) (layer Edge.Cuts) (width 0.05))
   (gr_line (start 164.2 51.4) (end 165.8 51.4) (layer Edge.Cuts) (width 0.05))
   (gr_line (start 164.2 53) (end 164.2 51.4) (layer Edge.Cuts) (width 0.05))
@@
   (gr_line (start 174.8 53) (end 174.8 147) (layer Edge.Cuts) (width 0.05))
   (gr_line (start 125.2 53) (end 134.2 53) (layer Edge.Cuts) (width 0.05))
-  (zone (net 0) (net_name "") (layer F.Cu) (hatch edge 0.508)
-    (connect_pads (clearance 0.508))
-    (min_thickness 0.254)
-    (fill yes (arc_segments 32) (thermal_gap 0.508) (thermal_bridge_width 0.508))
-    (polygon
-      (pts
-        (xy 186.8 39.5) (xy 179.3 155) (xy 118.3 154) (xy 106.8 38.5)
-      )
-    )
-  )
 )
