File: hardware/Side 1/Backup of not last minute bodged version/Side 1.kicad_pcb (KiCad board)
At the start: 2 copper layers, 126 x 214.2 mm, 4 parts

Commit message: God knows but a lot has changed
Other:
- board text added: "JLCJLCJLC"
